File: USB_Storage.kicad_sch (KiCad schematic)
At the start: 11 parts, among them J1 USB_A, U1 USBLC6-2SC6, U2 AP2112K-3.3, U3 GL3224-ONY

Commit message: 回路図の更新
Parts:
- added C10, C9: 18pF, symbol Device:C
- added C5, C7: 10uF, symbol Device:C
- added C6, C8: 0.1uF, symbol Device:C
- added R4: 12kΩ, symbol Device:R
- added U4: AP2112K-1.2, Package_TO_SOT_SMD:SOT-23-5, symbol Regulator_Linear:AP2112K-1.2
- added Y1: 25MHz, symbol Device:Crystal
Connections:
- net 3V3: now also C5.2, C6.2, U4.1 (VIN), U4.3 (EN)
- net GND: now also C10.2, C5.1, C6.1, C7.1, C8.2, C9.1, R4.1, U4.2 (GND)
- net at U3.13 (X1): now also C9.2, Y1.2
- net at U3.14 (X2): now also C10.1, Y1.1
- net at U3.16 (RTERM): now also R4.2
- net 1V2: now reaches U3.26 (DVDD12)
- net 1V2: now also U3.9 (AVDD12), C7.2, C8.1, U4.5 (VOUT)
