File: USB_Storage.kicad_sch (KiCad schematic)
At the start: 20 parts, among them J1 USB_A, U1 USBLC6-2SC6, U2 AP2112K-3.3, U3 GL3224-ONY, U4 AP2112K-1.2, Y1 25MHz

Commit message: 回路図の更新
Parts:
- added R_CLK, R_CMD, R_D0, R_D1, R_D2, R_D3: 0R, symbol Device:R
Connections:
- net EMMC_CLK: now also R_CLK.2; no longer U3.39 (S1CK_M1D0)
- net EMMC_CMD: now also R_CMD.1; no longer U3.40 (S1CM_M1D2)
- net EMMC_D0: now also R_D0.1; no longer U3.38 (S1D0_M1D1)
- net EMMC_D1: now also R_D1.1; no longer U3.37 (S1D1_M1BS)
- net EMMC_D2: now also R_D2.1; no longer U3.42 (S1D2_M1CK)
- net EMMC_D3: now also R_D3.1; no longer U3.41 (S1D3_M1D3)
- new net: R_D1.2, U3.37 (S1D1_M1BS)
- new net: R_D3.2, U3.41 (S1D3_M1D3)
- new net: R_D0.2, U3.38 (S1D0_M1D1)
- new net: R_D2.2, U3.42 (S1D2_M1CK)
- new net: R_CLK.1, U3.39 (S1CK_M1D0)
- new net: R_CMD.2, U3.40 (S1CM_M1D2)

Commit message: 回路図を更新しました
Parts:
- added R10, R6, R7, R8, R9: 47k, symbol Device:R
- added R11: 10k, symbol Device:R
- added U5: KLM8G1GETF-B041, KLMBG2JENB-B041_SAM, symbol KLM8G1GETF-B041_1:KLM8G1GETF-B041
Connections:
- net 3V3: now also R10.1, R11.2, R6.1, R7.1, R8.1, R9.1, U5.C6 (VCCQ), U5.E6 (VCC), U5.F5 (VCC), U5.K9 (VCC), U5.M4 (VCCQ), U5.N4 (VCCQ), U5.P3 (VCCQ), U5.P5 (VCCQ)
- net EMMC_CLK: now also U5.M6 (CLK)
- net EMMC_CMD: now also R6.2, U5.M5 (CMD)
- net EMMC_D0: now also R7.2, U5.A3 (DAT0)
- net EMMC_D1: now also R8.2, U5.A4 (DAT1)
- net EMMC_D2: now also R9.2, U5.A5 (DAT2)
- net EMMC_D3: now also R10.2, U5.B2 (DAT3)
- new net EMMC_RST_N: R11.1, U5.K5 (RSTN)
Other:
- moved on the sheet: C1, C10, C2, C3, C4, C5, C6, C7, C8, C9, J1, R1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

Commit message: 回路図の更新
Parts:
- added C11: 0.1µF, symbol Device:C
- added C12: 4.7µF, symbol Device:C
- added R12, R13: 0.1µF, symbol Device:R
- added R15: 1µF, symbol Device:R
Connections:
- net 3V3: now also C12.1; no longer U5.E6 (VCC), U5.F5 (VCC), U5.K9 (VCC)
- new net: R12.1, R13.1, R15.1
- new net: R13.2, U5.K9 (VCC)
- new net: C11.1, U5.E6 (VCC)
- new net: R12.2, U5.F5 (VCC)
- new net EMMC_VCC: C11.2, C12.2, R15.2

Commit message: 回路図の更新
Parts:
- removed R12: 0.1µF, symbol Device:R
- removed R15: 1µF, symbol Device:R
- added C13, C15, C16, C19, C20, C21, C22, C24: 0.1µF, symbol Device:C
- added C14, C18, C23: 1µF, symbol Device:C
- added C17, C25: 4.7µF, symbol Device:C
- added C26, C27: 0.1uF, symbol Device:C
- added C28, C29: 1uF, symbol Device:C
- C11: value 0.1µF -> 0.1uF
- C12: value 4.7µF -> 0.1uF
Connections:
- net EMMC_VCC is gone; now on net GND: C11.2, C12.2
- net 1V2: now also C26.1, C27.1, C29.2
- net 3V3: now also C11.1, R13.1, U5.E6 (VCC), U5.F5 (VCC), C13.2, C14.2, C15.2, C16.2, C17.1, C18.1, C19.2, C20.1, C21.1, C22.1, C23.1, C25.1, C28.2
- net GND: now also C13.1, C14.1, C15.1, C16.1, C17.2, C18.2, C19.1, C20.2, C21.2, C22.2, C23.2, C24.1, C25.2, C26.2, C27.2, C28.1, C29.1
- net at R13.2, U5.K9 (VCC): now also C24.2

Commit message: ERCのエラーの修正
Parts:
- added C30, C33: 1µF, symbol Device:C
- added C31, C32: 0.1µF, symbol Device:C
Connections:
- net GND: now also C30.2, C31.2, C32.2, C33.2
- net at U3.33 (VUHS_2): now also C32.1, C33.1
- net at U3.43 (VUHS_1): now also C30.1, C31.1
- no-connect marks 0 -> 25

Commit message: 回路図の更新
Parts:
- removed C5, C7: 10uF, symbol Device:C
- removed C6, C8: 0.1uF, symbol Device:C
- removed U4: AP2112K-1.2, Package_TO_SOT_SMD:SOT-23-5, symbol Regulator_Linear:AP2112K-1.2
- added C34: 1µF, symbol Device:C
- added C38: 10µF, symbol Device:C
- added C40: 4.7µF, symbol Device:C
- added C41, C44, C45, C46, C49: 0.1µF, symbol Device:C
- added C42: 1.0µF, symbol Device:C
- added C47, C48: 27pF, symbol Device:C
- added FB1: FerriteBead, symbol Device:FerriteBead
- added J2: USB_A, symbol Connector:USB_A
- added R12: 100kΩ, symbol Device:R
- added R14: 200kΩ, symbol Device:R
- added R5: 10kΩ, symbol Device:R
- added U4: USBLC6-2SC6, Package_TO_SOT_SMD:SOT-23-6, symbol Power_Protection:USBLC6-2SC6
- added U6: AP2112K-3.3, Package_TO_SOT_SMD:SOT-23-5, symbol Regulator_Linear:AP2112K-3.3
- added U8: AP2112K-1.8, Package_TO_SOT_SMD:SOT-23-5, symbol Regulator_Linear:AP2112K-1.8
- added U9: USB2642/ML, QFN48_7X7MC_MCH, symbol USB2642-ML:USB2642_ML
- added Y2: 24MHz, symbol Device:Crystal
- C10, C9: value 18pF -> 15pF
- C29: value 1uF -> 10µF
- R4: value 12kΩ -> 68Ω
Connections:
- net 3V3: now also C12.2; no longer C12.1
- net GND: now also C12.1, U5.A6 (VSS), U5.C4 (VSS), U5.E7 (VSS), U5.G5 (VSS), U5.K8 (VSS), U5.N2 (VSS), U5.N5 (VSS), U5.P4 (VSS), U5.P6 (VSS), C34.2, C38.2, C47.2, C48.1, C49.1, J2.4 (GND), R14.2, U4.2 (GND), U6.2 (GND), U8.2 (GND); no longer C12.2
- net USB_DP: now also J2.2 (D-), U4.3 (I/O2), U4.4 (I/O2), U9.42 (USBUP_DP)
- net at U5.C2 (VDDI): now also C34.1
- removed net 1V2: C26.1, C27.1, C29.2, U3.26 (DVDD12), U3.9 (AVDD12)
- new net: C48.2, U9.45 (XTAL1(CLKIN)), Y2.2
- new net: C40.1, C41.1, C44.1, C45.1, C46.1, R5.1, U6.5 (VOUT)
- new net: C44.2, U9.26 (VDD33)
- new net: C41.2, U9.12 (VDD33)
- new net: C45.2, U9.25 (VDD33)
- new net: C42.2, U9.15 (VDD18)
- new net: C40.2, U9.16 (VDD33)
- new net: C46.2, U9.34 (VDD33)
- new net: C49.2, R5.2, U9.38 (RESET_N)
- new net: R12.2, R14.1, U9.39 (VBUS_DET)
- new net: C47.1, U9.44 (XTAL2), Y2.1
- new net: C26.1, U3.26 (DVDD12)
- new net: C42.1, U8.5 (VOUT)
- new net: C27.1, U3.9 (AVDD12)
- new net USB_DM: J2.3 (D+), U4.1 (I/O1), U4.6 (I/O1), U9.43 (USBUP_DM)
- new net VBUS: FB1.1, J2.1 (VBUS), U4.5 (VBUS)
- new net VBUS_Filtered: C29.2, C38.1, FB1.2, R12.1, U6.1 (VIN), U6.3 (EN), U8.1 (VIN), U8.3 (EN)
- no-connect marks 25 -> 136
Other:
- moved on the sheet: C11, C12, C20

Commit message: 回路図の更新
Parts:
- removed C1, C3: 10uF, symbol Device:C
- removed C10, C9: 15pF, symbol Device:C
- removed C11, C12, C2, C26, C27, C4: 0.1uF, symbol Device:C
- removed C13, C15, C16, C19, C20, C21, C22, C24, C31, C32, C41: 0.1µF, symbol Device:C
- removed C14, C18, C23, C30, C33, C34: 1µF, symbol Device:C
- removed C17, C25, C40: 4.7µF, symbol Device:C
- removed C28: 1uF, symbol Device:C
- removed C29, C38: 10µF, symbol Device:C
- removed C42: 1.0µF, symbol Device:C
- removed C47, C48: 27pF, symbol Device:C
- removed J1: USB_A, symbol Connector:USB_A
- removed R1, R2, R3, R_CLK, R_CMD, R_D0, R_D1, R_D2, R_D3: 0R, symbol Device:R
- removed R10, R6, R7, R8, R9: 47k, symbol Device:R
- removed R11: 10k, symbol Device:R
- removed R13: 0.1µF, symbol Device:R
- removed R4: 68Ω, symbol Device:R
- removed R5: 10kΩ, symbol Device:R
- removed U1: USBLC6-2SC6, Package_TO_SOT_SMD:SOT-23-6, symbol Power_Protection:USBLC6-2SC6
- removed U2: AP2112K-3.3, Package_TO_SOT_SMD:SOT-23-5, symbol Regulator_Linear:AP2112K-3.3
- removed U3: GL3224-ONY, Package_DFN_QFN:QFN-48-1EP_7x7mm_P0.5mm_EP5.15x5.15mm, symbol Interface_USB:GL3224-ONY
- removed U5: KLM8G1GETF-B041, KLMBG2JENB-B041_SAM, symbol KLM8G1GETF-B041_1:KLM8G1GETF-B041
- removed U8: AP2112K-1.8, Package_TO_SOT_SMD:SOT-23-5, symbol Regulator_Linear:AP2112K-1.8
- removed Y1: 25MHz, symbol Device:Crystal
- removed Y2: 24MHz, symbol Device:Crystal
- added C35: 10µF, symbol Device:C
- added C43, C50, C51, C53, C54, C56, C61, C62, C63, C64, C66, C67, C68, C69, C71, C72, C73: 0.1µF, symbol Device:C
- added C52, C55, C60, C65: 4.7µF, symbol Device:C
- added C57: 1µF, symbol Device:C
- added C59, C75: 18pF, symbol Device:C
- added C70, C74: 1.0µF, symbol Device:C
- added FB2: FerriteBead, symbol Device:FerriteBead
- added R15: 100kΩ, symbol Device:R
- added R17: 12kΩ, symbol Device:R
- added R18: 1MΩ, symbol Device:R
- added U7: KLM8G1GETF-B041, KLMBG2JENB-B041_SAM, symbol KLM8G1GETF-B041_1:KLM8G1GETF-B041
- added Y3: 24MHz, symbol Device:Crystal
- C46: value 0.1µF -> 1.0µF
- R14: value 200kΩ -> 100kΩ
Connections:
- net GND: now also C44.2, C45.2, C46.2, U9.27 (TEST1), U9.28 (TEST2), U9.40 (TEST0), U9.49 (EPAD), C35.1, C43.2, C50.2, C51.2, C52.2, C53.2, C54.2, C55.2, C56.1, C57.2, C59.1, C60.2, C61.2, C62.2, C63.2, C64.2, C65.2, C66.2, C67.2, C68.2, C69.2, C70.2, C71.2, C72.2, C73.2, C74.2, C75.1, R15.2, R17.2, U7.A6 (VSS), U7.C4 (VSS), U7.E7 (VSS), U7.G5 (VSS), U7.H10 (VSS), U7.J5 (VSS), U7.K8 (VSS), U7.N2 (VSS), U7.N5 (VSS), U7.P4 (VSS), U7.P6 (VSS); no longer R14.2
- net VBUS_Filtered: now also C35.2, C57.1
- net at U9.45 (XTAL1(CLKIN)): now also C75.2, R18.2, Y3.2
- net at C44.1, U6.5 (VOUT): now also R14.1, U9.12 (VDD33), U9.16 (VDD33), U9.25 (VDD33), U9.26 (VDD33), U9.34 (VDD33), C53.1, C54.1, C55.1, C56.2, C60.1, C61.1, C62.1, C63.1, C64.1, C65.1, C66.1, C67.1, C68.1, C69.1, C72.1, FB2.2, U7.C6 (VCCQ), U7.E6 (VCC), U7.F5 (VCC), U7.J10 (VCC), U7.K9 (VCC), U7.M4 (VCCQ), U7.N4 (VCCQ), U7.P3 (VCCQ), U7.P5 (VCCQ); no longer C45.1, C46.1
- net at U9.15 (VDD18): now also C45.1, C46.1
- net at U9.17 (SD_D1): now also U7.A4 (DAT1)
- net at U9.18 (SD_D0): now also U7.A3 (DAT0)
- net at U9.21 (SD_CLK): now also U7.M6 (CLK)
- net at U9.24 (SD_CMD): now also U7.M5 (CMD)
- net at U9.32 (SD_D3): now also U7.B2 (DAT3)
- net at U9.33 (SD_D2): now also U7.A5 (DAT2)
- net at C49.2, U9.38 (RESET_N): now also R14.2
- net at R12.2, U9.39 (VBUS_DET): now also R15.1; no longer R14.1
- net at U9.41 (VDDA33): now also U9.48 (VDDA33), U9.5 (VDDA33), C43.1, C50.1, C51.1, C52.1, FB2.1
- net at U9.44 (XTAL2): now also C59.2, R18.1, Y3.1
- net at U9.46 (VDD18PLL): now also C73.1, C74.1
- net at U9.47 (RBIAS): now also R17.1
- new net: C70.1, C71.1, U7.C2 (VDDI)
- no-connect marks 136 -> 133
Other:
- moved on the sheet: C49, FB1, J2, R12, U4, U6, U9
