File: USB_Storage.kicad_sch (KiCad schematic)
At the start: 44 parts, among them J2 USB_A, U4 USBLC6-2SC6, U6 AP2112K-3.3, U7 KLM8G1GETF-B041, U9 USB2642/ML, Y3 24MHz

Commit message: 回路図の更新
Co-authored-by: Copilot <223556219+Copilot@users.noreply.github.com>
Parts:
- added R13, R16, R19, R20, R21, R22: 33Ω, Capacitor_SMD:C_1206_3216Metric_Pad1.33x1.80mm_HandSolder, symbol Device:R
- C35, C43, C44, C45, C46, C49, C50, C51, C52, C53, C54, C55, C56, C57, C59, C60, C61, C62, C63, C64, C65, C66, C67, C68, C69, C70, C71, C72, C73, C74, C75, FB1, FB2, R12, R14, R15, R17, R18: footprint (none) -> Capacitor_SMD:C_1206_3216Metric_Pad1.33x1.80mm_HandSolder
- J2: footprint (none) -> Connector_USB:USB_A_Molex_67643_Horizontal
- U7: footprint KLMBG2JENB-B041_SAM -> KLM8G1GETF-B041:KLMBG2JENB-B041_SAM
- U9: footprint QFN48_7X7MC_MCH -> USB2642:QFN48_7X7MC_MCH
- Y3: footprint (none) -> Crystal:Crystal_SMD_5032-2Pin_5.0x3.2mm_HandSoldering
Connections:
- net VBUS_Filtered is gone; now on net VBUS: C35.2, C57.1, FB1.2, R12.1, U6.1 (VIN), U6.3 (EN)
- net GND: now also J2.SH (Shield)
- net 3V3: now reaches C44.1, C53.1, C54.1, C55.1, C56.2, C60.1, C61.1, C62.1, C63.1, C64.1, C65.1, C66.1, C67.1, C68.1, C69.1, C72.1, FB2.2, R14.1, U6.5 (VOUT), U7.C6 (VCCQ), U7.E6 (VCC), U7.F5 (VCC), U7.J10 (VCC), U7.K9 (VCC), U7.M4 (VCCQ), U7.N4 (VCCQ), U7.P3 (VCCQ), U7.P5 (VCCQ), U9.12 (VDD33), U9.16 (VDD33), U9.25 (VDD33), U9.26 (VDD33), U9.34 (VDD33)
- net 3V3: now also C43.1, C50.1, C51.1, C52.1, FB2.1, U9.41 (VDDA33), U9.48 (VDDA33), U9.5 (VDDA33)
- net at U9.17 (SD_D1): now also R19.1; no longer U7.A4 (DAT1)
- net at U9.18 (SD_D0): now also R20.1; no longer U7.A3 (DAT0)
- net at U9.21 (SD_CLK): now also R16.2; no longer U7.M6 (CLK)
- net at U7.M5 (CMD): now also R13.1; no longer U9.24 (SD_CMD)
- net at U9.32 (SD_D3): now also R21.2; no longer U7.B2 (DAT3)
- net at U7.A5 (DAT2): now also R22.1; no longer U9.33 (SD_D2)
- net at C49.2, R14.2, U9.38 (RESET_N): now also U7.K5 (RSTN)
- new net: R19.2, U7.A4 (DAT1)
- new net: R13.2, U9.24 (SD_CMD)
- new net: R22.2, U9.33 (SD_D2)
- new net: R20.2, U7.A3 (DAT0)
- new net: R16.1, U7.M6 (CLK)
- new net: R21.1, U7.B2 (DAT3)
- no-connect marks 133 -> 146
Other:
- moved on the sheet: FB2
