File: USB_Storage.kicad_sch (KiCad schematic)
At the start: 50 parts, among them J2 USB_A, U4 USBLC6-2SC6, U6 AP2112K-3.3, U7 KLM8G1GETF-B041, U9 USB2642/ML, Y3 24MHz

Commit message: PCBレイアウトの更新
Changed lines of the file:
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@@
 					(size 1.27 1.27)
 				)
-				(justify right)
+				(justify left)
 			)
 		)
